Commit message: Improved UR5Robotiq
The old UR5Robotiq had trouble closing its gripper, because PyBullet handles mimic joints differently than Moveit or Gazebo.
Modified UR5Robotiq to use the models from here: https://github.com/ElectronicElephant/pybullet_ur5_robotiq,
which works nicely with PyBullet.

File: resources/ur5_robotiq.urdf (robot description, URDF)
Before this commit: robot ur5, 20 links, 19 joints
Links:
- removed link robotiq_85_base_link
- removed link robotiq_85_left_finger_link
- removed link robotiq_85_left_finger_tip_link
- removed link robotiq_85_left_inner_knuckle_link
- removed link robotiq_85_left_knuckle_link
- removed link robotiq_85_right_finger_link
- removed link robotiq_85_right_finger_tip_link
- removed link robotiq_85_right_inner_knuckle_link
- removed link robotiq_85_right_knuckle_link
- added link left_inner_finger, mass 0.0104003125914103; collision mesh filename=package://pycram/resources/meshes/robots/robotiq_85/collisi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 scale=0.001 0.001 0.001; visual mesh filename=package://pycram/resources/meshes/robots/robotiq_85/visual/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 scale=0.001 0.001 0.001
- added link left_inner_finger_pad, mass 1.; collision box size=0.022 0.00635 0.0375; visual box size=0.022 0.00635 0.0375
- added link left_inner_knuckle, mass 0.0271177346495152; collision mesh filename=package://pycram/resources/meshes/robots/robotiq_85/collisi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 scale=0.001 0.001 0.001; visual mesh filename=package://pycram/resources/meshes/robots/robotiq_85/visual/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 scale=0.001 0.001 0.001
- added link left_outer_finger, mass 0.022614240507152; collision mesh filename=package://pycram/resources/meshes/robots/robotiq_85/collisi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 scale=0.001 0.001 0.001; visual mesh filename=package://pycram/resources/meshes/robots/robotiq_85/visual/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 scale=0.001 0.001 0.001
- added link left_outer_knuckle, mass 0.00853198276973456; collision mesh filename=package://pycram/resources/meshes/robots/robotiq_85/collisi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 scale=0.001 0.001 0.001; visual mesh filename=package://pycram/resources/meshes/robots/robotiq_85/visual/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 scale=0.001 0.001 0.001
- added link right_inner_finger, mass 0.0104003125914103; collision mesh filename=package://pycram/resources/meshes/robots/robotiq_85/collisi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 scale=0.001 0.001 0.001; visual mesh filename=package://pycram/resources/meshes/robots/robotiq_85/visual/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 scale=0.001 0.001 0.001
- added link right_inner_finger_pad, mass 1; collision box size=0.022 0.00635 0.0375; visual box size=0.022 0.00635 0.0375
- added link right_inner_knuckle, mass 0.0271177346495152; collision mesh filename=package://pycram/resources/meshes/robots/robotiq_85/collisi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 scale=0.001 0.001 0.001; visual mesh filename=package://pycram/resources/meshes/robots/robotiq_85/visual/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 scale=0.001 0.001 0.001
- added link right_outer_finger, mass 0.022614240507152; collision mesh filename=package://pycram/resources/meshes/robots/robotiq_85/collisi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 scale=0.001 0.001 0.001; visual mesh filename=package://pycram/resources/meshes/robots/robotiq_85/visual/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 scale=0.001 0.001 0.001
- added link right_outer_knuckle, mass 0.00853198276973456; collision mesh filename=package://pycram/resources/meshes/robots/robotiq_85/collisi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 scale=0.001 0.001 0.001; visual mesh filename=package://pycram/resources/meshes/robots/robotiq_85/visual/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 scale=0.001 0.001 0.001
- added link robotiq_arg2f_base_link, mass 0.22652; collision mesh filename=package://pycram/resources/meshes/robots/robotiq_85/collisi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; visual mesh filename=package://pycram/resources/meshes/robots/robotiq_85/visual/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 scale=0.001 0.001 0.001
- link base_link: geometry collision mesh filename=package://pycram/resources/meshes/robots/ur5/collision/base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; visual mesh filename=package://pycram/resources/meshes/robots/ur5/visual/base.dae
- link forearm_link: geometry collision mesh filename=package://pycram/resources/meshes/robots/ur5/collision/fore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; visual mesh filename=package://pycram/resources/meshes/robots/ur5/visual/forearm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
- link robotiq_coupler: geometry collision mesh filename=package://pycram/resources/meshes/robots/robotiq_85/robotiq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 scale=1 1 1; visual mesh filename=package://pycram/resources/meshes/robots/robotiq_85/robotiq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 scale=1 1 1
- link shoulder_link: geometry collision mesh filename=package://pycram/resources/meshes/robots/ur5/collision/shou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; visual mesh filename=package://pycram/resources/meshes/robots/ur5/visual/shoulde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
- link upper_arm_link: geometry collision mesh filename=package://pycram/resources/meshes/robots/ur5/collision/uppe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; visual mesh filename=package://pycram/resources/meshes/robots/ur5/visual/upperar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
- link wrist_1_link: geometry collision mesh filename=package://pycram/resources/meshes/robots/ur5/collision/wris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; visual mesh filename=package://pycram/resources/meshes/robots/ur5/visual/wrist1.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
- link wrist_2_link: geometry collision mesh filename=package://pycram/resources/meshes/robots/ur5/collision/wris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; visual mesh filename=package://pycram/resources/meshes/robots/ur5/visual/wrist2.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
- link wrist_3_link: geometry collision mesh filename=package://pycram/resources/meshes/robots/ur5/collision/wris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; visual mesh filename=package://pycram/resources/meshes/robots/ur5/visual/wrist3.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
Joints:
- removed joint robotiq_85_left_finger_joint
- removed joint robotiq_85_left_finger_tip_joint
- removed joint robotiq_85_left_inner_knuckle_joint
- removed joint robotiq_85_left_knuckle_joint
- removed joint robotiq_85_right_finger_joint
- removed joint robotiq_85_right_finger_tip_joint
- removed joint robotiq_85_right_inner_knuckle_joint
- removed joint robotiq_85_right_knuckle_joint
- added joint finger_joint: type revolute, parent robotiq_arg2f_base_link, child left_outer_knuckle, origin xyz=0 -0.0306011 0.054904 rpy=0 0 3.14159265359, axis 1 0 0, limit lower=0 upper=0.8 effort=1000 velocity=2.0
- added joint left_inner_finger_joint: type revolute, parent left_outer_finger, child left_inner_finger, origin xyz=0 0.0061 0.0471 rpy=0 0 0, axis 1 0 0, limit lower=-0.8757 upper=0 effort=1000 velocity=2.0, mimic joint=finger_joint multiplier=-1 offset=0
- added joint left_inner_finger_pad_joint: type fixed, parent left_inner_finger, child left_inner_finger_pad, origin xyz=0 -0.0220203446692936 0.03242 rpy=0 0 0, axis 0 0 1
- added joint left_inner_knuckle_joint: type revolute, parent robotiq_arg2f_base_link, child left_inner_knuckle, origin xyz=0 -0.0127 0.06142 rpy=0 0 3.14159265359, axis 1 0 0, limit lower=0 upper=0.8757 effort=1000 velocity=2.0, mimic joint=finger_joint multiplier=1 offset=0
- added joint left_outer_finger_joint: type fixed, parent left_outer_knuckle, child left_outer_finger, origin xyz=0 0.0315 -0.0041 rpy=0 0 0, axis 1 0 0
- added joint right_inner_finger_joint: type revolute, parent right_outer_finger, child right_inner_finger, origin xyz=0 0.0061 0.0471 rpy=0 0 0, axis 1 0 0, limit lower=-0.8757 upper=0 effort=1000 velocity=2.0, mimic joint=finger_joint multiplier=-1 offset=0
- added joint right_inner_finger_pad_joint: type fixed, parent right_inner_finger, child right_inner_finger_pad, origin xyz=0 -0.0220203446692936 0.03242 rpy=0 0 0, axis 0 0 1
- added joint right_inner_knuckle_joint: type revolute, parent robotiq_arg2f_base_link, child right_inner_knuckle, origin xyz=0 0.0127 0.06142 rpy=0 0 0.0, axis 1 0 0, limit lower=0 upper=0.8757 effort=1000 velocity=2.0, mimic joint=finger_joint multiplier=1 offset=0
- added joint right_outer_finger_joint: type fixed, parent right_outer_knuckle, child right_outer_finger, origin xyz=0 0.0315 -0.0041 rpy=0 0 0, axis 1 0 0
- added joint right_outer_knuckle_joint: type revolute, parent robotiq_arg2f_base_link, child right_outer_knuckle, origin xyz=0 0.0306011 0.054904 rpy=0 0 0, axis 1 0 0, limit lower=0 upper=0.81 effort=1000 velocity=2.0, mimic joint=finger_joint multiplier=1 offset=0
- joint robotiq_85_base_joint: child robotiq_85_base_link -> robotiq_arg2f_base_link; origin xyz=0 0 0.004 rpy=0 -1.57079632679 3.14159265359 -> xyz=0 0 0.004 rpy=0 0 0
- joint robotiq_coupler_joint: origin xyz=0 0 0.004 rpy=0 0 -1.57079632679 -> xyz=0 0 0.004 rpy=0 0 0

Commit message: Fixes required after rebasing onto origin/dev

File: resources/ur5_robotiq.urdf (robot description, URDF)
Before this commit: robot ur5_robotiq, 22 links, 21 joints
Links:
- link base_link: geometry collision mesh filename=package://pycram/resources/meshes/ur5/collision/base.stl; visual mesh filename=package://pycram/resources/meshes/ur5/visual/base.dae
- link forearm_link: geometry collision mesh filename=package://pycram/resources/meshes/ur5/collision/forearm.stl; visual mesh filename=package://pycram/resources/meshes/ur5/visual/forearm.dae
- link left_inner_finger: geometry collision mesh filename=package://pycram/resources/meshes/robotiq_85/collision/robo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 scale=0.001 0.001 0.001; visual mesh filename=package://pycram/resources/meshes/robotiq_85/visual/robotiq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 scale=0.001 0.001 0.001
- link left_inner_knuckle: geometry collision mesh filename=package://pycram/resources/meshes/robotiq_85/collision/robo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 scale=0.001 0.001 0.001; visual mesh filename=package://pycram/resources/meshes/robotiq_85/visual/robotiq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 scale=0.001 0.001 0.001
- link left_outer_finger: geometry collision mesh filename=package://pycram/resources/meshes/robotiq_85/collision/robo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 scale=0.001 0.001 0.001; visual mesh filename=package://pycram/resources/meshes/robotiq_85/visual/robotiq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 scale=0.001 0.001 0.001
- link left_outer_knuckle: geometry collision mesh filename=package://pycram/resources/meshes/robotiq_85/collision/robo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 scale=0.001 0.001 0.001; visual mesh filename=package://pycram/resources/meshes/robotiq_85/visual/robotiq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 scale=0.001 0.001 0.001
- link right_inner_finger: geometry collision mesh filename=package://pycram/resources/meshes/robotiq_85/collision/robo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 scale=0.001 0.001 0.001; visual mesh filename=package://pycram/resources/meshes/robotiq_85/visual/robotiq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 scale=0.001 0.001 0.001
- link right_inner_knuckle: geometry collision mesh filename=package://pycram/resources/meshes/robotiq_85/collision/robo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 scale=0.001 0.001 0.001; visual mesh filename=package://pycram/resources/meshes/robotiq_85/visual/robotiq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 scale=0.001 0.001 0.001
- link right_outer_finger: geometry collision mesh filename=package://pycram/resources/meshes/robotiq_85/collision/robo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 scale=0.001 0.001 0.001; visual mesh filename=package://pycram/resources/meshes/robotiq_85/visual/robotiq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 scale=0.001 0.001 0.001
- link right_outer_knuckle: geometry collision mesh filename=package://pycram/resources/meshes/robotiq_85/collision/robo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 scale=0.001 0.001 0.001; visual mesh filename=package://pycram/resources/meshes/robotiq_85/visual/robotiq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 scale=0.001 0.001 0.001
- link robotiq_arg2f_base_link: geometry collision mesh filename=package://pycram/resources/meshes/robotiq_85/collision/robo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; visual mesh filename=package://pycram/resources/meshes/robotiq_85/visual/robotiq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 scale=0.001 0.001 0.001
- link robotiq_coupler: geometry collision mesh filename=package://pycram/resources/meshes/robotiq_85/robotiq_85_cou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 scale=1 1 1; visual mesh filename=package://pycram/resources/meshes/robotiq_85/robotiq_85_cou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 scale=1 1 1
- link shoulder_link: geometry collision mesh filename=package://pycram/resources/meshes/ur5/collision/shoulder.stl; visual mesh filename=package://pycram/resources/meshes/ur5/visual/shoulder.dae
- link upper_arm_link: geometry collision mesh filename=package://pycram/resources/meshes/ur5/collision/upperarm.stl; visual mesh filename=package://pycram/resources/meshes/ur5/visual/upperarm.dae
- link wrist_1_link: geometry collision mesh filename=package://pycram/resources/meshes/ur5/collision/wrist1.stl; visual mesh filename=package://pycram/resources/meshes/ur5/visual/wrist1.dae
- link wrist_2_link: geometry collision mesh filename=package://pycram/resources/meshes/ur5/collision/wrist2.stl; visual mesh filename=package://pycram/resources/meshes/ur5/visual/wrist2.dae
- link wrist_3_link: geometry collision mesh filename=package://pycram/resources/meshes/ur5/collision/wrist3.stl; visual mesh filename=package://pycram/resources/meshes/ur5/visual/wrist3.dae
